Commit message: Created core URDF

File: description/robot.urdf.xacro (robot description, xacro)
@@ -2,3 +2,7 @@
 <robot xmlns:xacro="http://www.ros.org/wiki/xacro"  name="robot">
     <xacro:include filename="robot_core.xacro" />
+    <xacro:include filename="gazebo_control.xacro" />
+    <xacro:include filename="lidar.xacro" />
+    <xacro:include filename="camera.xacro" />
+    <xacro:include filename="depth_camera.xacro" />
 </robot>

File: description/robot_core.xacro (robot description, xacro)
@@ -13,4 +13,7 @@
     <material name="black">
         <color rgba="0 0 0 1"/>
+    </material>
+    <material name="red">
+        <color rgba="1 0 0 1"/>
     </material>
     <link name="base_link">
@@ -40,4 +43,7 @@
         </xacro:inertial_box>
     </link>
+    <gazebo reference="chassis">
+        <material>Gazebo/White</material>
+    </gazebo>
     <!--LEFT WHEEL -->
     <joint name="left_wheel_joint" type="continuous">
@@ -63,4 +69,7 @@
         </xacro:inertial_cylinder>
     </link>
+    <gazebo reference="left_wheel">
+        <material>Gazebo/Blue</material>
+    </gazebo>
     <!-- RIGHT WHEEL -->
     <joint name="right_wheel_joint" type="continuous">
@@ -73,5 +82,5 @@
         <visual>
             <geometry>
-                <cylinder length="0.04" radius="0.05" />/>
+                <cylinder length="0.04" radius="0.05" />
             </geometry>
             <material name="blue"/>
@@ -79,5 +88,5 @@
         <collision>
             <geometry>
-                <cylinder length="0.04" radius="0.05" />/>
+                <cylinder length="0.04" radius="0.05" />
             </geometry>
         </collision>
@@ -86,4 +95,7 @@
         </xacro:inertial_cylinder>
     </link>
+    <gazebo reference="right_wheel">
+        <material>Gazebo/Blue</material>
+    </gazebo>
     <!-- CASTER WHEEL -->
     <joint name="caster_wheel_joint" type="fixed">
@@ -109,3 +121,8 @@
         </xacro:inertial_sphere>
     </link>
+    <gazebo reference="caster_wheel">
+        <material>Gazebo/Black</material>
+        <mu1 value="0.001"/>
+        <mu2 value="0.001"/>
+    </gazebo>
 </robot>
